Commit message: Add manually specified spheres

File: theseus/embodied/kinematics/tests/data/panda_no_gripper.urdf (robot description, URDF)
Before this commit: robot panda, 9 links, 8 joints
Links:
- link panda_link0: geometry collision mesh filename=meshes/collision/link0.stl; collision sphere radius=0.12
- link panda_link1: geometry collision mesh filename=meshes/collision/link1.stl; collision sphere radius=0.1
- link panda_link2: geometry collision mesh filename=meshes/collision/link2.stl; collision sphere radius=0.09
- link panda_link3: geometry collision mesh filename=meshes/collision/link3.stl; collision sphere radius=0.09
- link panda_link4: geometry collision mesh filename=meshes/collision/link4.stl; collision sphere radius=0.09
- link panda_link5: geometry collision mesh filename=meshes/collision/link5.stl; collision sphere radius=0.06
- link panda_link6: geometry collision mesh filename=meshes/collision/link6.stl; collision sphere radius=0.07
- link panda_link7: geometry collision mesh filename=meshes/collision/link7.stl; collision sphere radius=0.042
